File: dragon.kicad_pcb (KiCad board)
At the start: 2 copper layers, 57.2 x 53.3 mm, 17 parts, among them J2 Conn_01x08_Male, SW1 SW_Push, U1 ATtiny1614-SS

Commit message: Add files via upload
Other:
- board text added: "made by eri CC-BY-NC-SA"
- board text removed: "made by eri CC-BY-SA"
Changed lines of the file:
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@@
     (arrow2b (pts (xy 137.16 10.16) (xy 138.286504 9.573579)))
   )
-  (gr_text "made by eri\nCC-BY-SA" (at 165.735 33.655) (layer B.SilkS)
+  (gr_text "made by eri\nCC-BY-NC-SA" (at 165.735 33.655) (layer B.SilkS)
     (effects (font (size 1 1) (thickness 0.15)) (justify mirror))
   )
